File: hardware/brain/brain/brain.kicad_sch (KiCad schematic)
At the start: 0 parts

Commit message: wip: brain board revision — N16R8 MCU, AMS1117 LDO, 2x8 IDC, split schematic
Moves SD card-detect to GPIO 46, splits the brain schematic into audio,
interconnect, mcu, peripherals and power sheets, and adds TRRS protection
notes. Uncommitted work from April, parked as-is.

Co-Authored-By: Claude Opus 5.5 <noreply@anthropic.com>
Other:
- added sheet Audio (audio.kicad_sch)
- added sheet MCU (mcu.kicad_sch)
- added sheet Power (power.kicad_sch)
- added sheet Storage & Interconnect (peripherals.kicad_sch)
- company: (none) -> JP+ / mndxc
- title: (none) -> Stinger — Brain PCB (Core Engine)
